Commit message: Added mock hardware parameter and fixed udrf

File: src/roboguard_description/urdf/rove.base.ros2_control.urdf.xacro (robot description, xacro)
@@ -29,24 +29,28 @@
     </xacro:macro>
     <xacro:macro name="odrive_control" params="fl_id:=21 rl_id:=22 fr_id:=23 rr_id:=24">
-        <ros2_control name="odrive_control" type="system">
-            <hardware>
-                <plugin>odrive_hardware_interface_plugin/BetterODriveHardwareInterface</plugin>
-                <!-- <plugin>odrive_ros2_control_plugin/ODriveHardwareInterface</plugin> -->
-                <param name="can">can0</param>
-            </hardware>
-            <xacro:rove_odrive_motor suffix="fl" id="${fl_id}"/>
-            <xacro:rove_odrive_motor suffix="rl" id="${rl_id}"/>
-            <xacro:rove_odrive_motor suffix="fr" id="${fr_id}"/>
-            <xacro:rove_odrive_motor suffix="rr" id="${rr_id}"/>
-        </ros2_control>
-        <ros2_control name="fake_odrive_control" type="system">
-            <hardware>
-                <plugin>mock_components/GenericSystem</plugin>
-            </hardware>
-            <xacro:rove_fake_odrive_motor suffix="fl" id="${fl_id}"/>
-            <xacro:rove_fake_odrive_motor suffix="rl" id="${rl_id}"/>
-            <xacro:rove_fake_odrive_motor suffix="fr" id="${fr_id}"/>
-            <xacro:rove_fake_odrive_motor suffix="rr" id="${rr_id}"/>
-        </ros2_control>
+        <xacro:if value="${(fl_id != -1) and (rl_id != -1) and (fr_id != -1) and (rr_id != -1)}">
+            <ros2_control name="odrive_control" type="system">
+                <hardware>
+                    <plugin>odrive_hardware_interface_plugin/BetterODriveHardwareInterface</plugin>
+                    <!-- <plugin>odrive_ros2_control_plugin/ODriveHardwareInterface</plugin> -->
+                    <param name="can">can0</param>
+                </hardware>
+                <xacro:rove_odrive_motor suffix="fl" id="${fl_id}"/>
+                <xacro:rove_odrive_motor suffix="rl" id="${rl_id}"/>
+                <xacro:rove_odrive_motor suffix="fr" id="${fr_id}"/>
+                <xacro:rove_odrive_motor suffix="rr" id="${rr_id}"/>
+            </ros2_control>
+        </xacro:if>
+        <xacro:if value="${(fl_id == -1) or (rl_id == -1) or (fr_id == -1) or (rr_id == -1)}">
+            <ros2_control name="fake_odrive_control" type="system">
+                <hardware>
+                    <plugin>mock_components/GenericSystem</plugin>
+                </hardware>
+                <xacro:rove_fake_odrive_motor suffix="fl" id="${fl_id}"/>
+                <xacro:rove_fake_odrive_motor suffix="rl" id="${rl_id}"/>
+                <xacro:rove_fake_odrive_motor suffix="fr" id="${fr_id}"/>
+                <xacro:rove_fake_odrive_motor suffix="rr" id="${rr_id}"/>
+            </ros2_control>
+        </xacro:if>
     </xacro:macro>
 </robot>

File: src/roboguard_description/urdf/rove.base.urdf.xacro (robot description, xacro)
@@ -1,4 +1,5 @@
 <?xml version="1.0"?>
 <robot name="rove" xmlns:xacro="http://www.ros.org/wiki/xacro">
+    <xacro:arg name="use_mock_hardware" default="false"/>
     <material name="rubber_color">
         <color rgba="0.1 0.1 0.1 1.0" />
@@ -16,5 +17,5 @@
             <origin xyz="0 0 0" rpy="0 0 0" />
             <geometry>
-                <cube size="1 0.6 0.1" />
+                <box size="1 0.6 0.1" />
             </geometry>
             <material name="frame_color" />
@@ -23,5 +24,5 @@
             <origin xyz="0 0 0" rpy="0 0 0" />
             <geometry>
-                <cube size="1 0.6 0.1" />
+                <box size="1 0.6 0.1" />
             </geometry>
         </collision>
@@ -33,5 +34,9 @@
     </link>
     <!-- Put these at -1 to mock the motors if working without the motors -->
-    <!-- <xacro:odrive_control fl_id="21" rl_id="22" fr_id="23" rr_id="24" /> -->
-    <xacro:odrive_control fl_id="21" rl_id="-1" fr_id="-1" rr_id="-1" />
+    <xacro:if value="$(arg use_mock_hardware)">
+        <xacro:odrive_control fl_id="-1" rl_id="-1" fr_id="-1" rr_id="-1" />
+    </xacro:if>
+    <xacro:unless value="$(arg use_mock_hardware)">
+        <xacro:odrive_control fl_id="21" rl_id="22" fr_id="23" rr_id="24" />
+    </xacro:unless>
 </robot>

Commit message: Cleaned up useless comments Removed duplicate license files Removed old launch files Updated readme with accurate info Removed useless cmakelists tests Removed old config files Removed duplicate visual component in URDF Removed useless imports

File: src/roboguard_description/urdf/rove.base.ros2_control.urdf.xacro (robot description, xacro)
@@ -7,7 +7,9 @@
             <command_interface name="velocity"/>
             <command_interface name="effort"/>
+            <!-- NOT IMPLEMENTED -->
             <!-- <command_interface name="estop"/> -->
             <command_interface name="enable"/>
             <command_interface name="clear_errors_cmd"/>
+            <!-- UNTESTED -->
             <!-- <command_interface name="set_absolute_position"/> -->
             <state_interface name="position"/>
@@ -36,7 +38,9 @@
             <command_interface name="velocity"/>
             <command_interface name="effort"/>
+            <!-- NOT IMPLEMENTED -->
             <!-- <command_interface name="estop"/> -->
             <command_interface name="enable"/>
             <command_interface name="clear_errors_cmd"/>
+            <!-- UNTESTED -->
             <!-- <command_interface name="set_absolute_position"/> -->
             <state_interface name="position"/>
@@ -75,5 +79,4 @@
                 <hardware>
                     <plugin>odrive_hardware_interface_plugin/BetterODriveHardwareInterface</plugin>
-                    <!-- <plugin>odrive_ros2_control_plugin/ODriveHardwareInterface</plugin> -->
                     <param name="can">can0</param>
                 </hardware>

File: src/roboguard_description/urdf/rove.base.tracks.urdf.xacro (robot description, xacro)
@@ -28,11 +28,4 @@
         </joint>
         <link name="track_${suffix}">
-            <visual>
-                <origin xyz="0 0 0"/>
-                <geometry>
-                    <mesh filename="https://raw.githubusercontent.com/clubcapra/rove/main/src/rove_description/meshes/track.stl"/>
-                </geometry>
-                <material name="rubber_color" />
-            </visual>
             <visual>
                 <origin xyz="0 0 0" rpy="0 0 0"/>

File: src/roboguard_description/urdf/rove.base.urdf.xacro (robot description, xacro)
@@ -1,7 +1,12 @@
 <?xml version="1.0"?>
 <robot name="rove" xmlns:xacro="http://www.ros.org/wiki/xacro">
+    <!-- ODrive args -->
     <xacro:arg name="use_mock_odrives" default="false"/>
+    <xacro:arg name="can_channel" default="can0"/>
+    <!-- Ovis args -->
     <xacro:arg name="use_mock_ovis" default="false"/>
     <xacro:arg name="with_ovis" default="false"/>
+    <xacro:arg name="with_ovis" default="false"/>
+    <!-- TODO: Add ovis parameters (ip, etc) -->
     <material name="rubber_color">
         <color rgba="0.1 0.1 0.1 1.0" />
